File: usbcproto.sch (KiCad schematic (older format))
At the start: 26 parts, among them U1 STM32F103RETx, U2 MIC5219-3.3YM5, X1 PCB-USB-C, Y1 Crystal_GND2_Small

Commit message: Route pins and RGB LED.
Parts:
- added D1: FM-B2020RGBA-HG, fm-b2020rgba-hg:FM-B2020RGBA-HG, symbol fm-b2020rgba-hg:FM-B2020RGBA-HG
- added J1: Conn_01x04_Male, Connector_PinHeader_1.27mm:PinHeader_1x04_P1.27mm_Vertical, symbol Connector:Conn_01x04_Male
- added J2, J3: Conn_01x20_Male, Connector_PinHeader_1.27mm:PinHeader_1x20_P1.27mm_Vertical, symbol Connector:Conn_01x20_Male
Connections:
- net +3V3: now also D1.3 (+), J1.4 (Pin_4)
- net GND: now also J1.2 (Pin_2)
- net PC2: now reaches U1.10 (PC2)
- net PC2: now also J3.5 (Pin_5)
- net PC3: now reaches U1.11 (PC3)
- net PC3: now also J3.4 (Pin_4)
- net PA0: now reaches U1.14 (PA0)
- net PA0: now also J3.3 (Pin_3)
- net PA1: now reaches U1.15 (PA1)
- net PA1: now also J3.2 (Pin_2)
- net PA2: now reaches U1.16 (PA2)
- net PA2: now also J3.1 (Pin_1)
- net PA3: now reaches U1.17 (PA3)
- net PA3: now also J2.1 (Pin_1)
- net PC13: now reaches U1.2 (PC13)
- net PC13: now also J3.10 (Pin_10)
- net PA4: now reaches U1.20 (PA4)
- net PA4: now also J2.2 (Pin_2)
- net PA5: now reaches U1.21 (PA5)
- net PA5: now also J2.3 (Pin_3)
- net PA6: now reaches U1.22 (PA6)
- net PA6: now also J2.4 (Pin_4)
- net PA7: now reaches U1.23 (PA7)
- net PA7: now also J2.5 (Pin_5)
- net PC4: now reaches U1.24 (PC4)
- net PC4: now also J2.6 (Pin_6)
- net PC5: now reaches U1.25 (PC5)
- net PC5: now also J2.7 (Pin_7)
- net PB0: now reaches U1.26 (PB0)
- net PB0: now also J2.8 (Pin_8)
- net PB1: now reaches U1.27 (PB1)
- net PB1: now also J2.9 (Pin_9)
- net PB2: now reaches U1.28 (PB2)
- net PB2: now also J2.10 (Pin_10)
- net PB10: now reaches U1.29 (PB10)
- net PB10: now also J2.11 (Pin_11)
- net PC14: now reaches U1.3 (PC14)
- net PC14: now also J3.9 (Pin_9)
- net PB11: now reaches U1.30 (PB11)
- net PB11: now also J2.12 (Pin_12)
- net PB12: now reaches U1.33 (PB12)
- net PB12: now also J2.13 (Pin_13)
- net PB13: now reaches U1.34 (PB13)
- net PB13: now also J2.14 (Pin_14)
- net PB14: now reaches U1.35 (PB14)
- net PB14: now also J2.15 (Pin_15)
- net PB15: now reaches U1.36 (PB15)
- net PB15: now also J2.16 (Pin_16)
- net PC6: now reaches U1.37 (PC6)
- net PC6: now also J2.17 (Pin_17)
- net PC7: now reaches U1.38 (PC7)
- net PC7: now also J2.18 (Pin_18)
- net PC8: now reaches U1.39 (PC8)
- net PC8: now also J2.19 (Pin_19)
- net PC15: now reaches U1.4 (PC15)
- net PC15: now also J3.8 (Pin_8)
- net PC9: now reaches U1.40 (PC9)
- net PC9: now also J2.20 (Pin_20)
- net PA8: now reaches U1.41 (PA8)
- net PA8: now also D1.1 (R-)
- net PA9: now reaches U1.42 (PA9)
- net PA9: now also D1.4 (G-)
- net PA10: now reaches U1.43 (PA10)
- net PA10: now also D1.2 (B-)
- net SWDIO: now reaches U1.46 (PA13)
- net SWDIO: now also J1.1 (Pin_1)
- net SWCLK: now reaches U1.49 (PA14)
- net SWCLK: now also J1.3 (Pin_3)
- net PA15: now reaches U1.50 (PA15)
- net PC10: now reaches U1.51 (PC10)
- net PC11: now reaches U1.52 (PC11)
- net PC11: now also J3.20 (Pin_20)
- net PC12: now reaches U1.53 (PC12)
- net PC12: now also J3.19 (Pin_19)
- net PD2: now reaches U1.54 (PD2)
- net PD2: now also J3.18 (Pin_18)
- net PB3: now reaches U1.55 (PB3)
- net PB3: now also J3.17 (Pin_17)
- net PB4: now reaches U1.56 (PB4)
- net PB4: now also J3.16 (Pin_16)
- net PB5: now reaches U1.57 (PB5)
- net PB5: now also J3.15 (Pin_15)
- net PB6: now reaches U1.58 (PB6)
- net PB6: now also J3.14 (Pin_14)
- net PB7: now reaches U1.59 (PB7)
- net PB7: now also J3.13 (Pin_13)
- net PB8: now reaches U1.61 (PB8)
- net PB8: now also J3.12 (Pin_12)
- net PB9: now reaches U1.62 (PB9)
- net PB9: now also J3.11 (Pin_11)
- net PC0: now reaches U1.8 (PC0)
- net PC0: now also J3.7 (Pin_7)
- net PC1: now reaches U1.9 (PC1)
- net PC1: now also J3.6 (Pin_6)
Other:
- moved on the sheet: Y1
